File: CanSat_Upper/CanSat_Upper.kicad_sch (KiCad schematic)
At the start: 45 parts, among them J1 SERVO1, J10 Power GND, J2 SERVO1, J3 SERVO1, J4 SERVO1, J5 SERVO1, J6 SERVO1, J7 Power 5V, J8 JST_SH_10pin, J9 JST_SH_8pin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

Commit message: version 1.1 done
Parts:
- removed C12, C13: 1u, Capacitor_SMD:C_0603_1608Metric, symbol Device:C
- removed U6: TPS77033PDBV, Package_TO_SOT_SMD:SOT-23-5, symbol Regulator_Linear:TPS77033PDBV
- added D3: 5V_YELLOW, Diode_SMD:D_0805_2012Metric, symbol Device:LED
- added D4: 3V3_1_BLUE, Diode_SMD:D_0805_2012Metric, symbol Device:LED
- added D5: 3V3_2_BLUE, Diode_SMD:D_0805_2012Metric, symbol Device:LED
- added D6: GPS_GREEN, Diode_SMD:D_0805_2012Metric, symbol Device:LED
- R2, R3, R5, R6: value 0 -> RD; footprint Resistor_SMD:R_0603_1608Metric -> Capacitor_SMD:C_0603_1608Metric; LCSC C95177 -> (none)
Connections:
- net +3.3V3 is gone; now on net TIMEPULSE: R6.1
- net +3.3V: now also R3.1; no longer R2.1
- net +3.3V2: now also C8.1, C9.1, U1.13 (DVDD), U1.2 (AVDD)
- net +5V: now also R2.1
- net GND: now also D3.1 (K), D4.1 (K), D5.1 (K), D6.1 (K)
- net TIMEPULSE: now reaches U3.20 (TIMEPULSE)
- new net: D3.2 (A), R2.2
- new net: D5.2 (A), R5.2
- new net: D6.2 (A), R6.2
- new net: D4.2 (A), R3.2
- no-connect marks 30 -> 29
Other:
- note added: "4mA max"
- note added: "Diodes"
